File: DesignTest.kicad_pcb (KiCad board)
At the start: 2 copper layers, 36.6 x 31 mm, 6 parts, among them J1 Conn_01x02, J2 Conn_01x09, J3 Conn_01x04, J4 Conn_01x02, U1 4051

Commit message: development - added text to PCB
Other:
- board text added: "Development !"
Changed lines of the file:
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@@
     (area 103.556999 69.520999 140.283001 100.659001)
     (thickness 1.6)
-    (drawings 4)
+    (drawings 5)
     (tracks 76)
     (zones 0)
@@
     )
   )
+  (gr_text "Development !" (at 121.92 103.124) (layer F.SilkS)
+    (effects (font (size 1.5 1.5) (thickness 0.3)))
+  )
   (gr_line (start 103.632 100.584) (end 103.632 69.596) (angle 90) (layer Edge.Cuts) (width 0.15))

Commit message: Ready to go
Other:
- board text added: "Ready to go"
- board text removed: "Development !"
Changed lines of the file:
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@@
     (links 20)
     (no_connects 1)
-    (area 103.556999 69.520999 140.283001 100.659001)
+    (area 103.524999 69.520999 140.315001 104.474)
     (thickness 1.6)
     (drawings 5)
@@
     (aux_axis_origin 103.632 100.584)
     (grid_origin 115.824 65.024)
-    (visible_elements FFFFFF7F)
+    (visible_elements 7FFFFFFF)
     (pcbplotparams
       (layerselection 0x00030_80000001)
@@
     )
   )
-  (gr_text "Development !" (at 121.92 103.124) (layer F.SilkS)
+  (gr_text "Ready to go" (at 121.92 103.124) (layer F.SilkS)
     (effects (font (size 1.5 1.5) (thickness 0.3)))
   )
@@
   (segment (start 120.904 85.344) (end 120.904 78.74) (width 0.25) (layer F.Cu) (net 2))
   (segment (start 120.523 85.725) (end 120.904 85.344) (width 0.25) (layer F.Cu) (net 2))
-  (segment (start 118.745 83.185) (end 119.761 83.185) (width 0.25) (layer F.Cu) (net 3) (status 400000))
+  (segment (start 118.745 83.185) (end 119.761 83.185) (width 0.25) (layer F.Cu) (net 3))
   (segment (start 125.984 81.28) (end 129.54 81.28) (width 0.25) (layer B.Cu) (net 3))
   (segment (start 123.952 83.312) (end 125.984 81.28) (width 0.25) (layer B.Cu) (net 3))
@@
   (segment (start 119.38 84.328) (end 119.888 84.328) (width 0.25) (layer B.Cu) (net 5))
   (segment (start 117.348 82.296) (end 119.38 84.328) (width 0.25) (layer B.Cu) (net 5))
-  (segment (start 118.745 81.915) (end 117.221 81.915) (width 0.25) (layer F.Cu) (net 5) (status 400000))
+  (segment (start 118.745 81.915) (end 117.221 81.915) (width 0.25) (layer F.Cu) (net 5))
   (segment (start 127.508 84.328) (end 129.54 86.36) (width 0.25) (layer B.Cu) (net 5))
   (segment (start 119.888 84.328) (end 127.508 84.328) (width 0.25) (layer B.Cu) (net 5))
